File: hardware/COL_DRV.sch (KiCad schematic (older format))
At the start: 6 parts

Commit message: Add footprints to all symbols
Parts:
- C?: footprint (none) -> Capacitor_SMD:C_0402_1005Metric
- U?: footprint (none) -> waf:QFN-16_EP_2.5x2.5_Pitch0.4mm
Changed lines of the file:
@@
 $Descr A4 11693 8268
 encoding utf-8
-Sheet 42 44
+Sheet 41 44
 Title ""
 Date ""
@@
 F 0 "U?" H 4100 3500 50  0000 C CNN
 F 1 "SN74HC595B" H 4800 3500 50  0000 C CNN
-F 2 "" H 4050 3450 50  0001 C CNN
+F 2 "waf:QFN-16_EP_2.5x2.5_Pitch0.4mm" H 4050 3450 50  0001 C CNN
 F 3 "http://www.ti.com/lit/gpn/sn74hc595b" H 4050 3450 50  0001 C CNN
 	1    4500 2900
@@
 F 0 "C?" H 4115 1596 50  0000 L CNN
 F 1 "100n" H 4115 1505 50  0000 L CNN
-F 2 "" H 4038 1400 50  0001 C CNN
+F 2 "Capacitor_SMD:C_0402_1005Metric" H 4038 1400 50  0001 C CNN
 F 3 "~" H 4000 1550 50  0001 C CNN
 	1    4000 1550
@@
 P 4000 1800
 AR Path="/5CC10402/5D4CD97D" Ref="#PWR?"  Part="1"
-AR Path="/5CC10402/5D4C59DD/5D4CD97D" Ref="#PWR?"  Part="1"
-AR Path="/5CC10402/63C61482/5D4CD97D" Ref="#PWR?"  Part="1"
-AR Path="/5CC10402/64215E83/5D4CD97D" Ref="#PWR?"  Part="1"
-AR Path="/5CC10402/647DA0F2/5D4CD97D" Ref="#PWR?"  Part="1"
-F 0 "#PWR?" H 4000 1550 50  0001 C CNN
+AR Path="/5CC10402/5D4C59DD/5D4CD97D" Ref="#PWR0150"  Part="1"
+AR Path="/5CC10402/63C61482/5D4CD97D" Ref="#PWR0161"  Part="1"
+AR Path="/5CC10402/64215E83/5D4CD97D" Ref="#PWR0172"  Part="1"
+AR Path="/5CC10402/647DA0F2/5D4CD97D" Ref="#PWR0183"  Part="1"
+F 0 "#PWR0150" H 4000 1550 50  0001 C CNN
 F 1 "GND" H 4005 1627 50  0000 C CNN
 F 2 "" H 4000 1800 50  0001 C CNN
@@
 P 4000 1200
 AR Path="/5CC10402/5D4CD983" Ref="#PWR?"  Part="1"
-AR Path="/5CC10402/5D4C59DD/5D4CD983" Ref="#PWR?"  Part="1"
-AR Path="/5CC10402/63C61482/5D4CD983" Ref="#PWR?"  Part="1"
-AR Path="/5CC10402/64215E83/5D4CD983" Ref="#PWR?"  Part="1"
-AR Path="/5CC10402/647DA0F2/5D4CD983" Ref="#PWR?"  Part="1"
-F 0 "#PWR?" H 4000 1050 50  0001 C CNN
+AR Path="/5CC10402/5D4C59DD/5D4CD983" Ref="#PWR0151"  Part="1"
+AR Path="/5CC10402/63C61482/5D4CD983" Ref="#PWR0162"  Part="1"
+AR Path="/5CC10402/64215E83/5D4CD983" Ref="#PWR0173"  Part="1"
+AR Path="/5CC10402/647DA0F2/5D4CD983" Ref="#PWR0184"  Part="1"
+F 0 "#PWR0151" H 4000 1050 50  0001 C CNN
 F 1 "+BATT" H 4015 1373 50  0000 C CNN
 F 2 "" H 4000 1200 50  0001 C CNN
@@
 P 4500 3600
 AR Path="/5CC10402/5D4CD98F" Ref="#PWR?"  Part="1"
-AR Path="/5CC10402/5D4C59DD/5D4CD98F" Ref="#PWR?"  Part="1"
-AR Path="/5CC10402/63C61482/5D4CD98F" Ref="#PWR?"  Part="1"
-AR Path="/5CC10402/64215E83/5D4CD98F" Ref="#PWR?"  Part="1"
-AR Path="/5CC10402/647DA0F2/5D4CD98F" Ref="#PWR?"  Part="1"
-F 0 "#PWR?" H 4500 3350 50  0001 C CNN
+AR Path="/5CC10402/5D4C59DD/5D4CD98F" Ref="#PWR0152"  Part="1"
+AR Path="/5CC10402/63C61482/5D4CD98F" Ref="#PWR0163"  Part="1"
+AR Path="/5CC10402/64215E83/5D4CD98F" Ref="#PWR0174"  Part="1"
+AR Path="/5CC10402/647DA0F2/5D4CD98F" Ref="#PWR0185"  Part="1"
+F 0 "#PWR0152" H 4500 3350 50  0001 C CNN
 F 1 "GND" H 4505 3427 50  0000 C CNN
 F 2 "" H 4500 3600 50  0001 C CNN
@@
 P 8200 1300
 AR Path="/5CC10402/5E09784A" Ref="#PWR?"  Part="1"
-AR Path="/5CC10402/5D4C59DD/5E09784A" Ref="#PWR?"  Part="1"
-AR Path="/5CC10402/63C61482/5E09784A" Ref="#PWR?"  Part="1"
-AR Path="/5CC10402/64215E83/5E09784A" Ref="#PWR?"  Part="1"
-AR Path="/5CC10402/647DA0F2/5E09784A" Ref="#PWR?"  Part="1"
-F 0 "#PWR?" H 8200 1150 50  0001 C CNN
+AR Path="/5CC10402/5D4C59DD/5E09784A" Ref="#PWR0153"  Part="1"
+AR Path="/5CC10402/63C61482/5E09784A" Ref="#PWR0164"  Part="1"
+AR Path="/5CC10402/64215E83/5E09784A" Ref="#PWR0175"  Part="1"
+AR Path="/5CC10402/647DA0F2/5E09784A" Ref="#PWR0186"  Part="1"
+F 0 "#PWR0153" H 8200 1150 50  0001 C CNN
 F 1 "+BATT" H 8215 1473 50  0000 C CNN
 F 2 "" H 8200 1300 50  0001 C CNN
@@
 P 9800 2000
 AR Path="/5CC10402/5E09D225" Ref="#PWR?"  Part="1"
-AR Path="/5CC10402/5D4C59DD/5E09D225" Ref="#PWR?"  Part="1"
-AR Path="/5CC10402/63C61482/5E09D225" Ref="#PWR?"  Part="1"
-AR Path="/5CC10402/64215E83/5E09D225" Ref="#PWR?"  Part="1"
-AR Path="/5CC10402/647DA0F2/5E09D225" Ref="#PWR?"  Part="1"
-F 0 "#PWR?" H 9800 1850 50  0001 C CNN
+AR Path="/5CC10402/5D4C59DD/5E09D225" Ref="#PWR0154"  Part="1"
+AR Path="/5CC10402/63C61482/5E09D225" Ref="#PWR0165"  Part="1"
+AR Path="/5CC10402/64215E83/5E09D225" Ref="#PWR0176"  Part="1"
+AR Path="/5CC10402/647DA0F2/5E09D225" Ref="#PWR0187"  Part="1"
+F 0 "#PWR0154" H 9800 1850 50  0001 C CNN
 F 1 "+BATT" H 9815 2173 50  0000 C CNN
 F 2 "" H 9800 2000 50  0001 C CNN
@@
 P 8200 2500
 AR Path="/5CC10402/5E0A73E9" Ref="#PWR?"  Part="1"
-AR Path="/5CC10402/5D4C59DD/5E0A73E9" Ref="#PWR?"  Part="1"
-AR Path="/5CC10402/63C61482/5E0A73E9" Ref="#PWR?"  Part="1"
-AR Path="/5CC10402/64215E83/5E0A73E9" Ref="#PWR?"  Part="1"
-AR Path="/5CC10402/647DA0F2/5E0A73E9" Ref="#PWR?"  Part="1"
-F 0 "#PWR?" H 8200 2350 50  0001 C CNN
+AR Path="/5CC10402/5D4C59DD/5E0A73E9" Ref="#PWR0155"  Part="1"
+AR Path="/5CC10402/63C61482/5E0A73E9" Ref="#PWR0166"  Part="1"
+AR Path="/5CC10402/64215E83/5E0A73E9" Ref="#PWR0177"  Part="1"
+AR Path="/5CC10402/647DA0F2/5E0A73E9" Ref="#PWR0188"  Part="1"
+F 0 "#PWR0155" H 8200 2350 50  0001 C CNN
 F 1 "+BATT" H 8215 2673 50  0000 C CNN
 F 2 "" H 8200 2500 50  0001 C CNN
@@
 P 9800 3200
 AR Path="/5CC10402/5E0A73F9" Ref="#PWR?"  Part="1"
-AR Path="/5CC10402/5D4C59DD/5E0A73F9" Ref="#PWR?"  Part="1"
-AR Path="/5CC10402/63C61482/5E0A73F9" Ref="#PWR?"  Part="1"
-AR Path="/5CC10402/64215E83/5E0A73F9" Ref="#PWR?"  Part="1"
-AR Path="/5CC10402/647DA0F2/5E0A73F9" Ref="#PWR?"  Part="1"
-F 0 "#PWR?" H 9800 3050 50  0001 C CNN
+AR Path="/5CC10402/5D4C59DD/5E0A73F9" Ref="#PWR0156"  Part="1"
+AR Path="/5CC10402/63C61482/5E0A73F9" Ref="#PWR0167"  Part="1"
+AR Path="/5CC10402/64215E83/5E0A73F9" Ref="#PWR0178"  Part="1"
+AR Path="/5CC10402/647DA0F2/5E0A73F9" Ref="#PWR0189"  Part="1"
+F 0 "#PWR0156" H 9800 3050 50  0001 C CNN
 F 1 "+BATT" H 9815 3373 50  0000 C CNN
 F 2 "" H 9800 3200 50  0001 C CNN
@@
 P 8200 3700
 AR Path="/5CC10402/5E0AD314" Ref="#PWR?"  Part="1"
-AR Path="/5CC10402/5D4C59DD/5E0AD314" Ref="#PWR?"  Part="1"
-AR Path="/5CC10402/63C61482/5E0AD314" Ref="#PWR?"  Part="1"
-AR Path="/5CC10402/64215E83/5E0AD314" Ref="#PWR?"  Part="1"
-AR Path="/5CC10402/647DA0F2/5E0AD314" Ref="#PWR?"  Part="1"
-F 0 "#PWR?" H 8200 3550 50  0001 C CNN
+AR Path="/5CC10402/5D4C59DD/5E0AD314" Ref="#PWR0157"  Part="1"
+AR Path="/5CC10402/63C61482/5E0AD314" Ref="#PWR0168"  Part="1"
+AR Path="/5CC10402/64215E83/5E0AD314" Ref="#PWR0179"  Part="1"
+AR Path="/5CC10402/647DA0F2/5E0AD314" Ref="#PWR0190"  Part="1"
+F 0 "#PWR0157" H 8200 3550 50  0001 C CNN
 F 1 "+BATT" H 8215 3873 50  0000 C CNN
 F 2 "" H 8200 3700 50  0001 C CNN
@@
 P 9800 4400
 AR Path="/5CC10402/5E0AD324" Ref="#PWR?"  Part="1"
-AR Path="/5CC10402/5D4C59DD/5E0AD324" Ref="#PWR?"  Part="1"
-AR Path="/5CC10402/63C61482/5E0AD324" Ref="#PWR?"  Part="1"
-AR Path="/5CC10402/64215E83/5E0AD324" Ref="#PWR?"  Part="1"
-AR Path="/5CC10402/647DA0F2/5E0AD324" Ref="#PWR?"  Part="1"
-F 0 "#PWR?" H 9800 4250 50  0001 C CNN
+AR Path="/5CC10402/5D4C59DD/5E0AD324" Ref="#PWR0158"  Part="1"
+AR Path="/5CC10402/63C61482/5E0AD324" Ref="#PWR0169"  Part="1"
+AR Path="/5CC10402/64215E83/5E0AD324" Ref="#PWR0180"  Part="1"
+AR Path="/5CC10402/647DA0F2/5E0AD324" Ref="#PWR0191"  Part="1"
+F 0 "#PWR0158" H 9800 4250 50  0001 C CNN
 F 1 "+BATT" H 9815 4573 50  0000 C CNN
 F 2 "" H 9800 4400 50  0001 C CNN
@@
 P 8200 4900
 AR Path="/5CC10402/5E0AD33C" Ref="#PWR?"  Part="1"
-AR Path="/5CC10402/5D4C59DD/5E0AD33C" Ref="#PWR?"  Part="1"
-AR Path="/5CC10402/63C61482/5E0AD33C" Ref="#PWR?"  Part="1"
-AR Path="/5CC10402/64215E83/5E0AD33C" Ref="#PWR?"  Part="1"
-AR Path="/5CC10402/647DA0F2/5E0AD33C" Ref="#PWR?"  Part="1"
-F 0 "#PWR?" H 8200 4750 50  0001 C CNN
+AR Path="/5CC10402/5D4C59DD/5E0AD33C" Ref="#PWR0159"  Part="1"
+AR Path="/5CC10402/63C61482/5E0AD33C" Ref="#PWR0170"  Part="1"
+AR Path="/5CC10402/64215E83/5E0AD33C" Ref="#PWR0181"  Part="1"
+AR Path="/5CC10402/647DA0F2/5E0AD33C" Ref="#PWR0192"  Part="1"
+F 0 "#PWR0159" H 8200 4750 50  0001 C CNN
 F 1 "+BATT" H 8215 5073 50  0000 C CNN
 F 2 "" H 8200 4900 50  0001 C CNN
@@
 P 9800 5600
 AR Path="/5CC10402/5E0AD34C" Ref="#PWR?"  Part="1"
-AR Path="/5CC10402/5D4C59DD/5E0AD34C" Ref="#PWR?"  Part="1"
-AR Path="/5CC10402/63C61482/5E0AD34C" Ref="#PWR?"  Part="1"
-AR Path="/5CC10402/64215E83/5E0AD34C" Ref="#PWR?"  Part="1"
-AR Path="/5CC10402/647DA0F2/5E0AD34C" Ref="#PWR?"  Part="1"
-F 0 "#PWR?" H 9800 5450 50  0001 C CNN
+AR Path="/5CC10402/5D4C59DD/5E0AD34C" Ref="#PWR0160"  Part="1"
+AR Path="/5CC10402/63C61482/5E0AD34C" Ref="#PWR0171"  Part="1"
+AR Path="/5CC10402/64215E83/5E0AD34C" Ref="#PWR0182"  Part="1"
+AR Path="/5CC10402/647DA0F2/5E0AD34C" Ref="#PWR0193"  Part="1"
+F 0 "#PWR0160" H 9800 5450 50  0001 C CNN
 F 1 "+BATT" H 9815 5773 50  0000 C CNN
 F 2 "" H 9800 5600 50  0001 C CNN
