File: hardware/LEDS.sch (KiCad schematic (older format))
At the start: 0 parts

Commit message: Add LED column and instanciate 32 of them
Parts:
- added C?: 100n, symbol Device:C
- added C?: 47u, symbol Device:C
- added C?: 470u, symbol Device:C
- added R?: R, symbol Device:R
- added U?: TLC59581, Package_DFN_QFN:QFN-56-1EP_8x8mm_P0.5mm_EP5.6x5.6mm_ThermalVias, symbol waf:TLC59581
Connections:
- new net: R?.1, U?.1 (IREF)
- new net: R?.2, U?.56 (IREFGND)
- new net +BATT: C?.1, C?.1, C?.1, U?.43 (VCC)
- new net B0: U?.10 (OUTB0)
- new net B1: U?.13 (OUTB1)
- new net B10: U?.46 (OUTB10)
- new net B11: U?.49 (OUTB11)
- new net B12: U?.52 (OUTB12)
- new net B13: U?.55 (OUTB13)
- new net B14: U?.4 (OUTB14)
- new net B15: U?.7 (OUTB15)
- new net B2: U?.16 (OUTB2)
- new net B3: U?.19 (OUTB3)
- new net B4: U?.22 (OUTB4)
- new net B5: U?.25 (OUTB5)
- new net B6: U?.32 (OUTB6)
- new net B7: U?.35 (OUTB7)
- new net B8: U?.38 (OUTB8)
- new net B9: U?.41 (OUTB9)
- new net G0: U?.9 (OUTG0)
- new net G1: U?.12 (OUTG1)
- new net G10: U?.45 (OUTG10)
- new net G11: U?.48 (OUTG11)
- new net G12: U?.51 (OUTG12)
- new net G13: U?.54 (OUTG13)
- new net G14: U?.3 (OUTG14)
- new net G15: U?.6 (OUTG15)
- new net G2: U?.15 (OUTG2)
- new net G3: U?.18 (OUTG3)
- new net G4: U?.21 (OUTG4)
- new net G5: U?.24 (OUTG5)
- new net G6: U?.31 (OUTG6)
- new net G7: U?.34 (OUTG7)
- new net G8: U?.37 (OUTG8)
- new net G9: U?.40 (OUTG9)
- new net GCLK: U?.29 (GCLK)
- new net GND: C?.2, C?.2, C?.2, U?.57 (GND)
- new net LAT: U?.27 (LAT)
- new net R0: U?.8 (OUTR0)
- new net R1: U?.11 (OUTR1)
- new net R10: U?.44 (OUTR10)
- new net R11: U?.47 (OUTR11)
- new net R12: U?.50 (OUTR12)
- new net R13: U?.53 (OUTR13)
- new net R14: U?.2 (OUTR14)
- new net R15: U?.5 (OUTR15)
- new net R2: U?.14 (OUTR2)
- new net R3: U?.17 (OUTR3)
- new net R4: U?.20 (OUTR4)
- new net R5: U?.23 (OUTR5)
- new net R6: U?.30 (OUTR6)
- new net R7: U?.33 (OUTR7)
- new net R8: U?.36 (OUTR8)
- new net R9: U?.39 (OUTR9)
- new net SCLK: U?.28 (SCLK)
- new net SIN: U?.26 (SIN)
- new net SOUT: U?.42 (SOUT)
Other:
- note removed: "https://www.mouser.fr/ProductDetail/Inolux/IN-B101FCH"

Commit message: Add shift registers and first mosfet
Parts:
- added C? (x4): 100n, symbol Device:C
- added Q?: NTJD4152PT1GOSCT-ND, Package_TO_SOT_SMD:SOT-363_SC-70-6, symbol waf:NTJD4152PT1GOSCT-ND
- added TP?: COL_SER_OUT, symbol Connector:TestPoint
- added U? (x4): SN74HC595B, symbol waf:SN74HC595B
Connections:
- net +BATT: now also C?.1, C?.1, C?.1, C?.1, U?.16 (Vcc), U?.16 (Vcc), U?.16 (Vcc), U?.16 (Vcc)
- net GND: now also C?.2, C?.2, C?.2, C?.2, U?.8 (GND), U?.8 (GND), U?.8 (GND), U?.8 (GND)
- new net: U?.14 (SER), U?.9 (QH') (x3)
- new net: TP?.1, U?.9 (QH')
- new net COL_0: U?.15 (QA)
- new net COL_1: U?.1 (QB)
- new net COL_10: U?.2 (QC)
- new net COL_11: U?.3 (QD)
- new net COL_12: U?.4 (QE)
- new net COL_13: U?.5 (QF)
- new net COL_14: U?.6 (QG)
- new net COL_15: U?.7 (QH)
- new net COL_16: U?.15 (QA)
- new net COL_17: U?.1 (QB)
- new net COL_18: U?.2 (QC)
- new net COL_19: U?.3 (QD)
- new net COL_2: U?.2 (QC)
- new net COL_20: U?.4 (QE)
- new net COL_21: U?.5 (QF)
- new net COL_22: U?.6 (QG)
- new net COL_23: U?.7 (QH)
- new net COL_24: U?.15 (QA)
- new net COL_25: U?.1 (QB)
- new net COL_26: U?.2 (QC)
- new net COL_27: U?.3 (QD)
- new net COL_28: U?.4 (QE)
- new net COL_29: U?.5 (QF)
- new net COL_3: U?.3 (QD)
- new net COL_30: U?.6 (QG)
- new net COL_31: U?.7 (QH)
- new net COL_4: U?.4 (QE)
- new net COL_5: U?.5 (QF)
- new net COL_6: U?.6 (QG)
- new net COL_7: U?.7 (QH)
- new net COL_8: U?.15 (QA)
- new net COL_9: U?.1 (QB)
- new net COL_RCLK: U?.12 (RCLK), U?.12 (RCLK), U?.12 (RCLK), U?.12 (RCLK)
- new net COL_SER: U?.14 (SER)
- new net COL_SRCLK: U?.11 (SRCLK), U?.11 (SRCLK), U?.11 (SRCLK), U?.11 (SRCLK)
- new net COL_nOE: U?.13 (nOE), U?.13 (nOE), U?.13 (nOE), U?.13 (nOE)
- new net COL_nSRCLR: U?.10 (nSRCLR), U?.10 (nSRCLR), U?.10 (nSRCLR), U?.10 (nSRCLR)

Commit message: Add LEDs column drivers
Parts:
- removed C? (x4): 100n, symbol Device:C
- removed Q?: NTJD4152PT1GOSCT-ND, Package_TO_SOT_SMD:SOT-363_SC-70-6, symbol waf:NTJD4152PT1GOSCT-ND
- removed U? (x4): SN74HC595B, symbol waf:SN74HC595B
Connections:
- net Column driver 3/COL_SER_OUT: now reaches TP?.1
Other:
- moved on the sheet: C?, R?, TP?, U?

Commit message: Add footprints to all symbols
Parts:
- C?: footprint (none) -> Capacitor_SMD:C_0402_1005Metric
- C?: footprint (none) -> Capacitor_SMD:C_0603_1608Metric_Pad1.05x0.95mm_HandSolder
- C?: footprint (none) -> Capacitor_SMD:CP_Elec_10x10.5
- R?: footprint (none) -> Resistor_SMD:R_0603_1608Metric_Pad1.05x0.95mm_HandSolder
Changed lines of the file:
@@
 F 0 "C?" H 1715 5196 50  0000 L CNN
 F 1 "100n" H 1715 5105 50  0000 L CNN
-F 2 "" H 1638 5000 50  0001 C CNN
+F 2 "Capacitor_SMD:C_0402_1005Metric" H 1638 5000 50  0001 C CNN
 F 3 "~" H 1600 5150 50  0001 C CNN
 	1    1600 5150
@@
 F 0 "C?" H 1315 5196 50  0000 L CNN
 F 1 "47u" H 1315 5105 50  0000 L CNN
-F 2 "" H 1238 5000 50  0001 C CNN
+F 2 "Capacitor_SMD:C_0603_1608Metric_Pad1.05x0.95mm_HandSolder" H 1238 5000 50  0001 C CNN
 F 3 "~" H 1200 5150 50  0001 C CNN
 	1    1200 5150
@@
 	1600 5400 1600 5300
 $Comp
-L power:GND #PWR?
+L power:GND #PWR0146
 U 1 1 5C81AEEE
 P 1200 5500
-F 0 "#PWR?" H 1200 5250 50  0001 C CNN
+F 0 "#PWR0146" H 1200 5250 50  0001 C CNN
 F 1 "GND" H 1205 5327 50  0000 C CNN
 F 2 "" H 1200 5500 50  0001 C CNN
@@
 	1200 4900 1200 4800
 $Comp
-L power:+BATT #PWR?
+L power:+BATT #PWR0147
 U 1 1 5C81C613
 P 1200 4800
-F 0 "#PWR?" H 1200 4650 50  0001 C CNN
+F 0 "#PWR0147" H 1200 4650 50  0001 C CNN
 F 1 "+BATT" H 1215 4973 50  0000 C CNN
 F 2 "" H 1200 4800 50  0001 C CNN
@@
 F 0 "C?" H 915 5196 50  0000 L CNN
 F 1 "470u" H 915 5105 50  0000 L CNN
-F 2 "" H 838 5000 50  0001 C CNN
+F 2 "Capacitor_SMD:CP_Elec_10x10.5" H 838 5000 50  0001 C CNN
 F 3 "~" H 800 5150 50  0001 C CNN
 	1    800  5150
@@
 	2100 6900 2100 6800
 $Comp
-L power:+BATT #PWR?
+L power:+BATT #PWR0148
 U 1 1 5C832749
 P 2100 6800
-F 0 "#PWR?" H 2100 6650 50  0001 C CNN
+F 0 "#PWR0148" H 2100 6650 50  0001 C CNN
 F 1 "+BATT" H 2115 6973 50  0000 C CNN
 F 2 "" H 2100 6800 50  0001 C CNN
@@
 	1900 12300 1900 12400
 $Comp
-L power:GND #PWR?
+L power:GND #PWR0149
 U 1 1 601C7944
 P 2100 12500
-F 0 "#PWR?" H 2100 12250 50  0001 C CNN
+F 0 "#PWR0149" H 2100 12250 50  0001 C CNN
 F 1 "GND" H 2105 12327 50  0000 C CNN
 F 2 "" H 2100 12500 50  0001 C CNN
@@
 F 0 "R?" H 1470 12096 50  0000 L CNN
 F 1 "R" H 1470 12005 50  0000 L CNN
-F 2 "" V 1330 12050 50  0001 C CNN
+F 2 "Resistor_SMD:R_0603_1608Metric_Pad1.05x0.95mm_HandSolder" V 1330 12050 50  0001 C CNN
 F 3 "~" H 1400 12050 50  0001 C CNN
 	1    1400 12050

Commit message: Add TXB0104 Level shifter for column drivers
Parts:
- added C?: 100n, Capacitor_SMD:C_0402_1005Metric, symbol Device:C
- added R?: 100k, Resistor_SMD:R_0603_1608Metric_Pad1.05x0.95mm_HandSolder, symbol Device:R
- added R?: R, Resistor_SMD:R_0603_1608Metric_Pad1.05x0.95mm_HandSolder, symbol Device:R
- added U?: TXB0104RUT, Package_DFN_QFN:Texas_R_PUQFN-N12, symbol Logic_LevelTranslator:TXB0104RUT
Connections:
- net +BATT: now also R?.1, U?.11 (VCCB); no longer C?.1, C?.1, C?.1, U?.43 (VCC)
- net COL_RCLK: now also U?.3 (A2), U?.9 (B2)
- net COL_SER: now also U?.4 (A3), U?.8 (B3)
- net COL_SRCLK: now also U?.10 (B1), U?.2 (A1)
- net COL_nOE: now also R?.1, U?.5 (A4), U?.7 (B4)
- net COL_nSRCLR: now also C?.1, R?.2
- net GND: now also C?.2, R?.2, U?.6 (GND)
- new net +3V3: C?.1, C?.1, C?.1, U?.1 (VCCA), U?.12 (OE), U?.43 (VCC)
Other:
- note added: "RC=10ms"
- moved on the sheet: TP?
