File: hardware/LED_COL.sch (KiCad schematic (older format))
At the start: 16 parts

Commit message: Add footprints to all symbols
Parts:
- D? (x16): footprint (none) -> waf:IN-B101FCH
Changed lines of the file:
@@
 $Descr A4 11693 8268
 encoding utf-8
-Sheet 9 44
+Sheet 33 44
 Title ""
 Date ""
@@
 F 0 "D?" H 2750 2797 50  0000 C CNN
 F 1 "LED_RGB" H 2750 2706 50  0000 C CNN
-F 2 "" H 2750 2250 50  0001 C CNN
+F 2 "waf:IN-B101FCH" H 2750 2250 50  0001 C CNN
 F 3 "https://www.mouser.fr/datasheet/2/180/IN-B101FCH-1488525.pdf" H 2750 2250 50  0001 C CNN
 	1    2700 2300
@@
 F 0 "D?" H 4750 5497 50  0000 C CNN
 F 1 "LED_RGB" H 4750 5406 50  0000 C CNN
-F 2 "" H 4750 4950 50  0001 C CNN
+F 2 "waf:IN-B101FCH" H 4750 4950 50  0001 C CNN
 F 3 "https://www.mouser.fr/datasheet/2/180/IN-B101FCH-1488525.pdf" H 4750 4950 50  0001 C CNN
 	1    4700 5000
@@
 F 0 "D?" H 4750 4597 50  0000 C CNN
 F 1 "LED_RGB" H 4750 4506 50  0000 C CNN
-F 2 "" H 4750 4050 50  0001 C CNN
+F 2 "waf:IN-B101FCH" H 4750 4050 50  0001 C CNN
 F 3 "https://www.mouser.fr/datasheet/2/180/IN-B101FCH-1488525.pdf" H 4750 4050 50  0001 C CNN
 	1    4700 4100
@@
 F 0 "D?" H 4750 3697 50  0000 C CNN
 F 1 "LED_RGB" H 4750 3606 50  0000 C CNN
-F 2 "" H 4750 3150 50  0001 C CNN
+F 2 "waf:IN-B101FCH" H 4750 3150 50  0001 C CNN
 F 3 "https://www.mouser.fr/datasheet/2/180/IN-B101FCH-1488525.pdf" H 4750 3150 50  0001 C CNN
 	1    4700 3200
@@
 F 0 "D?" H 4750 2797 50  0000 C CNN
 F 1 "LED_RGB" H 4750 2706 50  0000 C CNN
-F 2 "" H 4750 2250 50  0001 C CNN
+F 2 "waf:IN-B101FCH" H 4750 2250 50  0001 C CNN
 F 3 "https://www.mouser.fr/datasheet/2/180/IN-B101FCH-1488525.pdf" H 4750 2250 50  0001 C CNN
 	1    4700 2300
@@
 F 0 "D?" H 2750 5497 50  0000 C CNN
 F 1 "LED_RGB" H 2750 5406 50  0000 C CNN
-F 2 "" H 2750 4950 50  0001 C CNN
+F 2 "waf:IN-B101FCH" H 2750 4950 50  0001 C CNN
 F 3 "https://www.mouser.fr/datasheet/2/180/IN-B101FCH-1488525.pdf" H 2750 4950 50  0001 C CNN
 	1    2700 5000
@@
 F 0 "D?" H 2750 4597 50  0000 C CNN
 F 1 "LED_RGB" H 2750 4506 50  0000 C CNN
-F 2 "" H 2750 4050 50  0001 C CNN
+F 2 "waf:IN-B101FCH" H 2750 4050 50  0001 C CNN
 F 3 "https://www.mouser.fr/datasheet/2/180/IN-B101FCH-1488525.pdf" H 2750 4050 50  0001 C CNN
 	1    2700 4100
@@
 F 0 "D?" H 2750 3697 50  0000 C CNN
 F 1 "LED_RGB" H 2750 3606 50  0000 C CNN
-F 2 "" H 2750 3150 50  0001 C CNN
+F 2 "waf:IN-B101FCH" H 2750 3150 50  0001 C CNN
 F 3 "https://www.mouser.fr/datasheet/2/180/IN-B101FCH-1488525.pdf" H 2750 3150 50  0001 C CNN
 	1    2700 3200
@@
 F 0 "D?" H 6750 2797 50  0000 C CNN
 F 1 "LED_RGB" H 6750 2706 50  0000 C CNN
-F 2 "" H 6750 2250 50  0001 C CNN
+F 2 "waf:IN-B101FCH" H 6750 2250 50  0001 C CNN
 F 3 "https://www.mouser.fr/datasheet/2/180/IN-B101FCH-1488525.pdf" H 6750 2250 50  0001 C CNN
 	1    6700 2300
@@
 F 0 "D?" H 8750 5497 50  0000 C CNN
 F 1 "LED_RGB" H 8750 5406 50  0000 C CNN
-F 2 "" H 8750 4950 50  0001 C CNN
+F 2 "waf:IN-B101FCH" H 8750 4950 50  0001 C CNN
 F 3 "https://www.mouser.fr/datasheet/2/180/IN-B101FCH-1488525.pdf" H 8750 4950 50  0001 C CNN
 	1    8700 5000
@@
 F 0 "D?" H 8750 4597 50  0000 C CNN
 F 1 "LED_RGB" H 8750 4506 50  0000 C CNN
-F 2 "" H 8750 4050 50  0001 C CNN
+F 2 "waf:IN-B101FCH" H 8750 4050 50  0001 C CNN
 F 3 "https://www.mouser.fr/datasheet/2/180/IN-B101FCH-1488525.pdf" H 8750 4050 50  0001 C CNN
 	1    8700 4100
@@
 F 0 "D?" H 8750 3697 50  0000 C CNN
 F 1 "LED_RGB" H 8750 3606 50  0000 C CNN
-F 2 "" H 8750 3150 50  0001 C CNN
+F 2 "waf:IN-B101FCH" H 8750 3150 50  0001 C CNN
 F 3 "https://www.mouser.fr/datasheet/2/180/IN-B101FCH-1488525.pdf" H 8750 3150 50  0001 C CNN
 	1    8700 3200
@@
 F 0 "D?" H 8750 2797 50  0000 C CNN
 F 1 "LED_RGB" H 8750 2706 50  0000 C CNN
-F 2 "" H 8750 2250 50  0001 C CNN
+F 2 "waf:IN-B101FCH" H 8750 2250 50  0001 C CNN
 F 3 "https://www.mouser.fr/datasheet/2/180/IN-B101FCH-1488525.pdf" H 8750 2250 50  0001 C CNN
 	1    8700 2300
@@
 F 0 "D?" H 6750 5497 50  0000 C CNN
 F 1 "LED_RGB" H 6750 5406 50  0000 C CNN
-F 2 "" H 6750 4950 50  0001 C CNN
+F 2 "waf:IN-B101FCH" H 6750 4950 50  0001 C CNN
 F 3 "https://www.mouser.fr/datasheet/2/180/IN-B101FCH-1488525.pdf" H 6750 4950 50  0001 C CNN
 	1    6700 5000
@@
 F 0 "D?" H 6750 4597 50  0000 C CNN
 F 1 "LED_RGB" H 6750 4506 50  0000 C CNN
-F 2 "" H 6750 4050 50  0001 C CNN
+F 2 "waf:IN-B101FCH" H 6750 4050 50  0001 C CNN
 F 3 "https://www.mouser.fr/datasheet/2/180/IN-B101FCH-1488525.pdf" H 6750 4050 50  0001 C CNN
 	1    6700 4100
@@
 F 0 "D?" H 6750 3697 50  0000 C CNN
 F 1 "LED_RGB" H 6750 3606 50  0000 C CNN
-F 2 "" H 6750 3150 50  0001 C CNN
+F 2 "waf:IN-B101FCH" H 6750 3150 50  0001 C CNN
 F 3 "https://www.mouser.fr/datasheet/2/180/IN-B101FCH-1488525.pdf" H 6750 3150 50  0001 C CNN
 	1    6700 3200
