File: hardware/NFC.sch (KiCad schematic (older format))
At the start: 46 parts

Commit message: Add footprints to all symbols
Parts:
- C? (x17): footprint (none) -> Capacitor_SMD:C_0402_1005Metric
- C? (x4): footprint (none) -> Capacitor_SMD:C_0805_2012Metric_Pad1.15x1.40mm_HandSolder
- C? (x4): footprint (none) -> Capacitor_SMD:C_0603_1608Metric_Pad1.05x0.95mm_HandSolder
- L? (x2): footprint (none) -> Inductor_SMD:L_0402_1005Metric
- R? (x5): footprint (none) -> Resistor_SMD:R_0402_1005Metric
- R? (x2): footprint (none) -> Resistor_SMD:R_0603_1608Metric_Pad1.05x0.95mm_HandSolder
- U?: footprint (none) -> Package_DFN_QFN:QFN-40-1EP_6x6mm_P0.5mm_EP4.6x4.6mm
- Y?: footprint (none) -> Crystal:Crystal_SMD_HC49-SD_HandSoldering

Commit message: Place BQ25892
Parts:
- FB? (x2): footprint (none) -> Inductor_SMD:L_0603_1608Metric
Changed lines of the file:
@@
 F 0 "FB?" V 1276 5900 50  0000 C CNN
 F 1 "Ferrite_Bead" V 1367 5900 50  0000 C CNN
-F 2 "" V 1480 5900 50  0001 C CNN
+F 2 "Inductor_SMD:L_0603_1608Metric" V 1480 5900 50  0001 C CNN
 F 3 "~" H 1550 5900 50  0001 C CNN
 	1    1550 5900
@@
 F 0 "FB?" V 1276 3600 50  0000 C CNN
 F 1 "Ferrite_Bead" V 1367 3600 50  0000 C CNN
-F 2 "" V 1480 3600 50  0001 C CNN
+F 2 "Inductor_SMD:L_0603_1608Metric" V 1480 3600 50  0001 C CNN
 F 3 "~" H 1550 3600 50  0001 C CNN
 	1    1550 3600
