File: hardware/USB-C.sch (KiCad schematic (older format))
At the start: 9 parts

Commit message: Add footprints to all symbols
Parts:
- C? (x2): footprint (none) -> Capacitor_SMD:C_0402_1005Metric
- J?: footprint (none) -> Connector_USB:USB_C_Receptacle_Amphenol_12401610E4-2A
- R?: footprint (none) -> Resistor_SMD:R_0805_2012Metric_Pad1.15x1.40mm_HandSolder
- R? (x3): footprint (none) -> Resistor_SMD:R_0603_1608Metric_Pad1.05x0.95mm_HandSolder
- R?: footprint (none) -> Resistor_SMD:R_0402_1005Metric
Changed lines of the file:
@@
 $Descr A4 11693 8268
 encoding utf-8
-Sheet 3 44
+Sheet 2 44
 Title "WAF WAF Howling badge"
 Date ""
@@
 F 0 "C?" H 2325 6750 50  0000 L CNN
 F 1 "4.7nF" H 2325 6550 50  0000 L CNN
-F 2 "" H 2338 6500 50  0001 C CNN
+F 2 "Capacitor_SMD:C_0402_1005Metric" H 2338 6500 50  0001 C CNN
 F 3 "~" H 2300 6650 50  0001 C CNN
 	1    2300 6650
@@
 F 0 "R?" V 2080 6650 50  0000 C CNN
 F 1 "1M" V 2000 6650 50  0000 C CNN
-F 2 "" V 1930 6650 50  0001 C CNN
+F 2 "Resistor_SMD:R_0805_2012Metric_Pad1.15x1.40mm_HandSolder" V 1930 6650 50  0001 C CNN
 F 3 "~" H 2000 6650 50  0001 C CNN
 	1    2000 6650
@@
 F 0 "J?" H 2200 5850 50  0000 L CNN
 F 1 "USB_C_Receptacle" H 3000 5850 50  0000 R CNN
-F 2 "" H 2750 4700 50  0001 C CNN
+F 2 "Connector_USB:USB_C_Receptacle_Amphenol_12401610E4-2A" H 2750 4700 50  0001 C CNN
 F 3 "https://www.usb.org/sites/default/files/documents/usb_type-c.zip" H 2750 4700 50  0001 C CNN
 	1    2600 4700
@@
 F 0 "C?" H 8425 2650 50  0000 L CNN
 F 1 "100n" H 8425 2450 50  0000 L CNN
-F 2 "" H 8438 2400 50  0001 C CNN
+F 2 "Capacitor_SMD:C_0402_1005Metric" H 8438 2400 50  0001 C CNN
 F 3 "~" H 8400 2550 50  0001 C CNN
 	1    8400 2550
@@
 F 0 "R?" V 8980 3950 50  0000 C CNN
 F 1 "1K" V 8900 3950 50  0000 C CNN
-F 2 "" V 8830 3950 50  0001 C CNN
+F 2 "Resistor_SMD:R_0603_1608Metric_Pad1.05x0.95mm_HandSolder" V 8830 3950 50  0001 C CNN
 F 3 "~" H 8900 3950 50  0001 C CNN
 	1    8900 3950
@@
 F 0 "R?" V 9180 3850 50  0000 C CNN
 F 1 "DNP" V 9100 3850 50  0000 C CNN
-F 2 "" V 9030 3850 50  0001 C CNN
+F 2 "Resistor_SMD:R_0603_1608Metric_Pad1.05x0.95mm_HandSolder" V 9030 3850 50  0001 C CNN
 F 3 "~" H 9100 3850 50  0001 C CNN
 	1    9100 3850
@@
 F 0 "R?" V 7080 2650 50  0000 C CNN
 F 1 "R" V 7000 2650 50  0000 C CNN
-F 2 "" V 6930 2650 50  0001 C CNN
+F 2 "Resistor_SMD:R_0402_1005Metric" V 6930 2650 50  0001 C CNN
 F 3 "~" H 7000 2650 50  0001 C CNN
 	1    7000 2650
@@
 F 0 "R?" V 9130 3100 50  0000 C CNN
 F 1 "900K" V 9050 3100 50  0000 C CNN
-F 2 "" V 8980 3100 50  0001 C CNN
+F 2 "Resistor_SMD:R_0603_1608Metric_Pad1.05x0.95mm_HandSolder" V 8980 3100 50  0001 C CNN
 F 3 "~" H 9050 3100 50  0001 C CNN
 	1    9050 3100
